File: pcb/UltraHawk/UltraHawk.kicad_pcb (KiCad board)
At the start: 2 copper layers, 75 parts, among them J1 USB_C_Receptacle_USB2.0_14P, J10 Screw_Terminal_01x02, J11 Conn_01x03_Pin, J12 Conn_01x03_Pin, J13 Conn_01x03_Pin, J14 Conn_01x03_Pin, J15 Conn_01x03_Pin, J2 Conn_01x04_Pin, J3 Conn_01x03_Pin, J4 Conn_01x04_Pin, J5 Conn_01x04_Pin, J6 Conn_01x06_Pin, J7 Screw_Terminal_01x02, J8 Screw_Terminal_01x02, J9 Screw_Terminal_01x02, SW1 SW_SPDT, U1 STM32H723VGTx, U2 AMS1117-3.3, U3 BMI270, U4 BMP581, U5 LIS3MDL, U6 TPS565208, U7 AO3400A, U8 AO3400A, U9 AO3400A, Y1 16MHz

Commit message: Pcb layout
Parts:
- removed R4: 1k5, Resistor_SMD:R_0805_2012Metric
- added D2: GREEN, LED_SMD:LED_0805_2012Metric, F.Cu at (68.0, 124.4)
- added H1: MountingHole, MountingHole:MountingHole_3.2mm_M3, F.Cu at (51.8, 75.2)
- added H2: MountingHole, MountingHole:MountingHole_3.2mm_M3, F.Cu at (94.2, 75.2)
- added H3: MountingHole, MountingHole:MountingHole_3.2mm_M3, F.Cu at (94.0, 144.5)
- added H4: MountingHole, MountingHole:MountingHole_3.2mm_M3, F.Cu at (52.0, 144.5)
- added R17: 220, Resistor_SMD:R_0805_2012Metric, F.Cu at (68.0, 120.2)
- J1: value USB_C_Receptacle_USB2.0_14P -> USB_C_Receptacle_USB2.0_16P; footprint easyeda2kicad:USB-C_SMD-TYPE-C-31-M-12_1 -> Connector_USB:USB_C_Receptacle_GCT_USB4105-xx-A_16P_TopMnt_Horizontal
- SW1: value SW_SPDT -> TS-1088R-02026; footprint easyeda2kicad:SW-TH_SHOU-HAN_SS12D10G4 -> easyeda2kicad:SW-SMD_L3.9-W3.0-P4.45
- Y1: value 16MHz -> 16MHZ; footprint Crystal:Crystal_HC49-4H_Vertical -> Crystal:Crystal_HC49-U_Vertical
- moved J7 82.4 mm to (89.2, 130.8)
- moved J14 81.8 mm to (58.6, 132.8), turned to -90 degrees
- moved J2 80.5 mm to (53.4, 137.8), turned to 90 degrees
- moved U2 76.9 mm to (73.0, 130.3), turned to 90 degrees
- moved J13 76.2 mm to (58.6, 128.2), turned to -90 degrees
- moved C14 73.2 mm to (80.0, 139.0), turned to 90 degrees
- moved C26 71.9 mm to (83.5, 138.0), turned to -90 degrees
- moved C25 71.4 mm to (83.5, 134.5), turned to 90 degrees
- moved J12 70.7 mm to (58.6, 123.6), turned to -90 degrees
- moved C29 68.1 mm to (82.8, 143.2)
- moved C27 68.0 mm to (86.5, 137.0)
- moved C15 65.5 mm to (67.5, 134.5)
- moved J11 65.4 mm to (58.6, 119.0), turned to -90 degrees
- moved C30 62.6 mm to (82.8, 140.8)
- moved C28 62.3 mm to (81.2, 134.5), turned to 90 degrees
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Connections:
- J1 pad A8: (no net) -> unconnected-(J1-SBU1-PadA8)
- J1 pad B8: (no net) -> unconnected-(J1-SBU2-PadB8)
- J11 pad 1: PWM5 -> PWM1
- J12 pad 1: PWM4 -> PWM2
- J14 pad 1: PWM2 -> PWM4
- J15 pad 1: PWM1 -> PWM5
- R1 pad 1: Net-(SW1-B) -> GND
- SW1 pad 1: GND -> 3.3V
- SW1 pad 2: Net-(SW1-B) -> Net-(U1-BOOT0)
- U1 pad 45: BARO_CS -> unconnected-(U1-PE15-Pad45)
- U1 pad 46: SPI2_SCK -> unconnected-(U1-PB10-Pad46)
- U1 pad 47: unconnected-(U1-PB11-Pad47) -> MAG_CS
- U1 pad 52: unconnected-(U1-PB13-Pad52) -> BARO_CS
- U1 pad 55: unconnected-(U1-PD8-Pad55) -> PYRO_3
- U1 pad 56: unconnected-(U1-PD9-Pad56) -> PYRO_2
- U1 pad 57: unconnected-(U1-PD10-Pad57) -> PYRO_1
- U1 pad 68: unconnected-(U1-PA9-Pad68) -> SPI2_SCK
- U1 pad 7: PYRO_1 -> unconnected-(U1-PC13-Pad7)
- U1 pad 8: PYRO_2 -> unconnected-(U1-PC14-Pad8)
- U1 pad 81: MAG_CS -> unconnected-(U1-PD0-Pad81)
- U1 pad 88: unconnected-(U1-PD7-Pad88) -> Net-(U1-PD7)
- U1 pad 9: PYRO_3 -> unconnected-(U1-PC15-Pad9)
- Y1 pad 2: GND -> Net-(U1-PH1)
Routing:
- net GND: track 0.00 -> 72.2 mm, vias 0 -> 4
- net LIPO_HIGH: track 0.00 -> 47.1 mm
- net 5V: track 0.00 -> 20.0 mm
- net Net-(J8-Pin_1): track 0.00 -> 16.5 mm
- net Net-(U6-SW): track 0.00 -> 16.1 mm
- net UART5_TX: track 0.00 -> 15.2 mm
- net UART5_RX: track 0.00 -> 13.3 mm
- net Net-(U1-BOOT0): track 0.00 -> 13.0 mm
- net Net-(U1-PH0): track 0.00 -> 11.6 mm
- net Net-(J9-Pin_1): track 0.00 -> 11.1 mm
- net PYRO_3: track 0.00 -> 10.4 mm, vias 0 -> 2
- net 3.3V: track 0.00 -> 9.12 mm
- net Net-(U1-PH1): track 0.00 -> 8.24 mm
- net Net-(J10-Pin_1): track 0.00 -> 7.55 mm
- net Net-(U5-C1): track 0.00 -> 6.56 mm
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