File: pcb/UltraHawk/UltraHawk.kicad_sch (KiCad schematic)
At the start: 52 parts, among them J1 USB_C_Receptacle_USB2.0_14P, J2 Conn_01x04_Pin, J3 Conn_01x02_Pin, SW1 SW_SPDT, U1 STM32H723VGTx, U2 AMS1117-3.3, U3 BMI270, U4 BMP581, U5 LIS3MDL, U6 TPS565208, Y1 16MHz

Commit message: Journal Update #3
Parts:
- removed J3: Conn_01x02_Pin, symbol Connector:Conn_01x02_Pin
- added J10, J7, J8, J9: Screw_Terminal_01x02, symbol Connector:Screw_Terminal_01x02
- added J11, J12, J13, J14, J15, J3: Conn_01x03_Pin, symbol Connector:Conn_01x03_Pin
- added J4, J5: Conn_01x04_Pin, symbol Connector:Conn_01x04_Pin
- added J6: Conn_01x06_Pin, symbol Connector:Conn_01x06_Pin
- added R10, R9: 4.7k, symbol Device:R
- added R11, R14, R16: 100, symbol Device:R
- added R12, R13, R15: 10k, symbol Device:R
- added U7, U8, U9: AO3400A, SOT-23-3L_AOS, symbol 2026-06-17_17-28-57:AO3400A
Connections:
- net 3.3V: now also J4.1 (Pin_1), J5.1 (Pin_1), J6.1 (Pin_1), R10.1, R9.1
- net 5V: now also J11.2 (Pin_2), J12.2 (Pin_2), J13.2 (Pin_2), J14.2 (Pin_2), J15.2 (Pin_2), J3.2 (Pin_2)
- net GND: now also J11.3 (Pin_3), J12.3 (Pin_3), J13.3 (Pin_3), J14.3 (Pin_3), J15.3 (Pin_3), J3.3 (Pin_3), J4.2 (Pin_2), J5.4 (Pin_4), J6.2 (Pin_2), J7.1 (Pin_1), R12.1, R13.1, R15.1, U7.2 (S), U8.2 (S), U9.2 (S)
- net LIPO_HIGH: now also J10.2 (Pin_2), J7.2 (Pin_2), J8.2 (Pin_2), J9.2 (Pin_2)
- net MAG_CS: now also U1.81 (PD0); no longer U1.44 (PE14)
- net SPI4_NSS: now reaches U1.3 (PE4)
- net SPI4_NSS: now also J6.6 (Pin_6)
- net SPI4_SCK: now reaches U1.42 (PE12)
- net SPI4_SCK: now also J6.3 (Pin_3)
- net SPI4_MISO: now reaches U1.43 (PE13)
- net SPI4_MISO: now also J6.5 (Pin_5)
- net PWM5: now reaches U1.61 (PD14)
- net PWM5: now also J11.1 (Pin_1)
- net PWM6: now reaches U1.62 (PD15)
- net PWM6: now also J3.1 (Pin_1)
- net PWM1: now reaches U1.63 (PC6)
- net PWM1: now also J15.1 (Pin_1)
- net PWM2: now reaches U1.64 (PC7)
- net PWM2: now also J14.1 (Pin_1)
- net PWM3: now reaches U1.65 (PC8)
- net PWM3: now also J13.1 (Pin_1)
- net PWM4: now reaches U1.66 (PC9)
- net PWM4: now also J12.1 (Pin_1)
- net PYRO_1: now reaches U1.7 (PC13)
- net PYRO_1: now also R11.1, R12.2
- net PYRO_2: now reaches U1.8 (PC14)
- net PYRO_2: now also R13.2, R14.1
- net UART5_TX: now reaches U1.80 (PC12)
- net UART5_TX: now also J5.3 (Pin_3)
- net UART5_RX: now reaches U1.83 (PD2)
- net UART5_RX: now also J5.2 (Pin_2)
- net PYRO_3: now reaches U1.9 (PC15)
- net PYRO_3: now also R15.2, R16.1
- net I2C4_SCL: now reaches U1.92 (PB6)
- net I2C4_SCL: now also J4.3 (Pin_3), R10.2
- net I2C4_SDA: now reaches U1.93 (PB7)
- net I2C4_SDA: now also J4.4 (Pin_4), R9.2
- new net: J10.1 (Pin_1), U9.3 (D)
- new net: R14.2, U8.1 (G)
- new net: J9.1 (Pin_1), U8.3 (D)
- new net: J8.1 (Pin_1), U7.3 (D)
- new net: R11.2, U7.1 (G)
- new net: R16.2, U9.1 (G)
- new net SPI4_MOSI: J6.4 (Pin_4), U1.44 (PE14)
Other:
- note added: "Mosfets"

Commit message: Journal Update #4
Parts:
- C1, C10, C11, C12, C13, C14, C15, C16, C17, C18, C19, C2, C20, C21, C22, C23, C24, C3, C4, C5, C6, C7, C8, C9: footprint (none) -> Capacitor_SMD:C_0805_2012Metric
- C25, C26, C27, C28, C29, C30: footprint Capacitor_SMD:C_0603_1608Metric -> Capacitor_SMD:C_0805_2012Metric
- D1: footprint (none) -> LED_SMD:LED_0805_2012Metric
- FB1, R1, R10, R11, R12, R13, R14, R15, R16, R2, R3, R4, R5, R9: footprint (none) -> Resistor_SMD:R_0805_2012Metric
- J1: footprint (none) -> easyeda2kicad:USB-C_SMD-TYPE-C-31-M-12_1
- J10, J7, J8, J9: footprint (none) -> TerminalBlock:TerminalBlock_MaiXu_MX126-5.0-02P_1x02_P5.00mm
- J11, J12, J13, J14, J15, J3: footprint (none) -> Connector_PinHeader_2.54mm:PinHeader_1x03_P2.54mm_Vertical
- J2, J4, J5: footprint (none) -> Connector_PinHeader_2.54mm:PinHeader_1x04_P2.54mm_Vertical
- J6: footprint (none) -> Connector_PinHeader_2.54mm:PinHeader_1x06_P2.54mm_Vertical
- R6, R7, R8: footprint Resistor_SMD:R_0603_1608Metric_Pad0.98x0.95mm_HandSolder -> Resistor_SMD:R_0805_2012Metric
- SW1: footprint (none) -> easyeda2kicad:SW-TH_SHOU-HAN_SS12D10G4
- U3: footprint BMI270_BOS -> bmi270:BMI270_BOS
- U4: footprint QFN10_BMP581_BOS -> bmp581:QFN10_BMP581_BOS
- U7, U8, U9: footprint SOT-23-3L_AOS -> ao34400a:SOT-23-3L_AOS
- Y1: footprint (none) -> Crystal:Crystal_HC49-4H_Vertical

Commit message: Pcb layout
Parts:
- removed J1: USB_C_Receptacle_USB2.0_14P, easyeda2kicad:USB-C_SMD-TYPE-C-31-M-12_1, symbol Connector:USB_C_Receptacle_USB2.0_14P
- removed R4: 1k5, Resistor_SMD:R_0805_2012Metric, symbol Device:R
- removed SW1: SW_SPDT, easyeda2kicad:SW-TH_SHOU-HAN_SS12D10G4, symbol Switch:SW_SPDT
- removed Y1: 16MHz, Crystal:Crystal_HC49-4H_Vertical, symbol Device:Crystal_GND24
- added D2: GREEN, LED_SMD:LED_0805_2012Metric, symbol Device:LED
- added H1, H2, H3, H4: MountingHole, MountingHole:MountingHole_3.2mm_M3, symbol Mechanical:MountingHole
- added J1: USB_C_Receptacle_USB2.0_16P, Connector_USB:USB_C_Receptacle_GCT_USB4105-xx-A_16P_TopMnt_Horizontal, symbol Connector:USB_C_Receptacle_USB2.0_16P
- added R17: 220, Resistor_SMD:R_0805_2012Metric, symbol Device:R
- added SW1: TS-1088R-02026, easyeda2kicad:SW-SMD_L3.9-W3.0-P4.45, symbol easyeda2kicad:TS-1088R-02026
- added Y1: 16MHZ, Crystal:Crystal_HC49-U_Vertical, symbol Device:Crystal
Connections:
- net 3.3V: now also SW1.1
- net 5V: now also J1.A4 (VBUS), J1.A9 (VBUS), J1.B4 (VBUS), J1.B9 (VBUS)
- net BARO_CS: now also U1.52 (PB13); no longer U1.45 (PE15)
- net D+: now also J1.A6 (D+), J1.B6 (D+)
- net D-: now also J1.A7 (D-), J1.B7 (D-)
- net GND: now also R1.1, D2.1 (K), J1.A1 (GND), J1.A12 (GND), J1.B1 (GND), J1.B12 (GND), J1.SH (SHIELD)
- net MAG_CS: now also U1.47 (PB11); no longer U1.81 (PD0)
- net PWM1: now also J11.1 (Pin_1); no longer J15.1 (Pin_1)
- net PWM2: now also J12.1 (Pin_1); no longer J14.1 (Pin_1)
- net PWM4: now also J14.1 (Pin_1); no longer J12.1 (Pin_1)
- net PWM5: now also J15.1 (Pin_1); no longer J11.1 (Pin_1)
- net PYRO_1: now also U1.57 (PD10); no longer U1.7 (PC13)
- net PYRO_2: now also U1.56 (PD9); no longer U1.8 (PC14)
- net PYRO_3: now also U1.55 (PD8); no longer U1.9 (PC15)
- net SPI2_SCK: now also U1.68 (PA9); no longer U1.46 (PB10)
- net at C12.1, U1.12 (PH0): now also Y1.1
- net at C13.1, U1.13 (PH1): now also Y1.2
- net at U1.88 (PD7): now also R17.2
- net at R1.2, U1.94 (BOOT0): now also SW1.2
- net at R2.2: now also J1.A5 (CC1)
- net at R3.2: now also J1.B5 (CC2)
- new net: D2.2 (A), R17.1
- no-connect marks 8 -> 10
Other:
- moved on the sheet: R1
