File: pcb/UltraHawk.kicad_sch (KiCad schematic)
At the start: 80 parts, among them J1 USB_C_Receptacle_USB2.0_16P, J10 Screw_Terminal_01x02, J11 Conn_01x03_Pin, J12 Conn_01x03_Pin, J13 Conn_01x03_Pin, J14 Conn_01x03_Pin, J15 Conn_01x03_Pin, J2 Conn_01x04_Pin, J3 Conn_01x03_Pin, J4 Conn_01x04_Pin, J5 Conn_01x04_Pin, J6 Conn_01x06_Pin, J7 Screw_Terminal_01x02, J8 Screw_Terminal_01x02, J9 Screw_Terminal_01x02, SW1 TS-1088R-02026, U1 STM32H723VGTx, U2 AMS1117-3.3, U3 BMI270, U4 BMP581, U5 LIS3MDL, U6 TPS565208, U7 AO3400A, U8 AO3400A, U9 AO3400A, Y1 16MHZ

Commit message: Journal Update #5
Connections:
- net SPI2_SCK: now also U1.46 (PB10); no longer U1.68 (PA9)

Commit message: Journal Update
Parts:
- removed R6: 10k, Resistor_SMD:R_0805_2012Metric, symbol Device:R
- C14: value C -> 1u
- C22: value 100n -> 1uf
- C27, C28: value 0.1µF -> 100n
- FB1: footprint Resistor_SMD:R_0805_2012Metric -> Resistor_SMD:R_0603_1608Metric_Pad0.98x0.95mm_HandSolder
- L1: footprint Inductor_SMD:L_0805_2012Metric -> easyeda2kicad:IND-SMD_L5.8-W5.2
Connections:
- net LIPO_HIGH: now also U6.5 (EN)
