File: pcb/UltraHawk.kicad_pcb (KiCad board)
At the start: 2 copper layers, 80 parts, among them J1 USB_C_Receptacle_USB2.0_16P, J10 Screw_Terminal_01x02, J11 Conn_01x03_Pin, J12 Conn_01x03_Pin, J13 Conn_01x03_Pin, J14 Conn_01x03_Pin, J15 Conn_01x03_Pin, J2 Conn_01x04_Pin, J3 Conn_01x03_Pin, J4 Conn_01x04_Pin, J5 Conn_01x04_Pin, J6 Conn_01x06_Pin, J7 Screw_Terminal_01x02, J8 Screw_Terminal_01x02, J9 Screw_Terminal_01x02, SW1 TS-1088R-02026, U1 STM32H723VGTx, U2 AMS1117-3.3, U3 BMI270, U4 BMP581, U5 LIS3MDL, U6 TPS565208, U7 AO3400A, U8 AO3400A, U9 AO3400A, Y1 16MHZ

Commit message: fixes
Parts:
- moved R15 0.68 mm to (61.2, 106.3)
Routing:
- net PYRO_3: track 10.4 -> 11.2 mm
- net GND: track 72.2 -> 72.7 mm
Other:
- board outline added: 50 x 77 mm
Changed lines of the file:
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@@
 	(footprint "Resistor_SMD:R_0805_2012Metric"
 		(layer "F.Cu")
-		(at 61.0875 107 -90)
+		(at 61.25 106.3375 -90)
 		(descr "Resistor SMD 0805 (2012 Metric), square (rectangular) end terminal, IPC-7351 nominal, (Body size source: IPC-SM-782 page 72, https://www.pcb-3d.com/wordpress/wp-content/uploads/ipc-sm-782a_amendment_1_and_2.pdf)")
 		(tags "resistor")
@@
 		(end 98 148.5)
 		(stroke
-			(width 0.2)
+			(width 0.05)
 			(type default)
 		)
 		(fill no)
-		(layer "F.Cu")
+		(layer "Edge.Cuts")
 	)
 	(segment
@@
 		(start 83.5 138.95)
 		(end 85.5 138.95)
-		(width 0.2)
-		(layer "F.Cu")
-		(net "GND")
-	)
-	(segment
-		(start 61.0875 106.0875)
-		(end 64.1125 106.0875)
 		(width 0.2)
 		(layer "F.Cu")
@@
 	)
 	(segment
+		(start 61.25 106.0875)
+		(end 61.25 105.425)
+		(width 0.2)
+		(layer "F.Cu")
+		(net "GND")
+	)
+	(segment
 		(start 68.45 134.5)
 		(end 69.495339 133.454661)
@@
 		(start 69.183864 131.95)
 		(end 70.688525 133.454661)
+		(width 0.2)
+		(layer "F.Cu")
+		(net "GND")
+	)
+	(segment
+		(start 61.25 106.0875)
+		(end 64.1125 106.0875)
 		(width 0.2)
 		(layer "F.Cu")
@@
 	)
 	(segment
+		(start 61.25 108)
+		(end 61.25 107.25)
+		(width 0.2)
+		(layer "F.Cu")
+		(net "PYRO_3")
+	)
+	(segment

Commit message: Journal Update #5
Parts:
- moved D2 36.8 mm to (84.5, 91.5), turned to 180 degrees
- moved R15 34.8 mm to (84.5, 132.2), turned to 180 degrees
- moved C6 33.7 mm to (77.0, 73.5), turned to 180 degrees
- moved R17 32.6 mm to (81.5, 90.5)
- moved C21 30.2 mm to (50.0, 97.5), turned to 180 degrees
- moved C24 27.2 mm to (51.5, 95.0), turned to 180 degrees
- moved C22 23.0 mm to (50.5, 103.5), turned to -90 degrees
- moved U5 20.1 mm to (53.5, 97.5), turned to -90 degrees
- moved U4 19.7 mm to (58.0, 97.5)
- moved U3 18.9 mm to (63.8, 97.3), turned to 180 degrees
- moved C23 18.1 mm to (53.0, 103.5), turned to -90 degrees
- moved R12 16.7 mm to (85.2, 106.2), turned to 180 degrees
- moved U7 15.5 mm to (85.2, 99.0), turned to 0 degrees
- moved R11 14.9 mm to (84.2, 103.2), turned to 90 degrees
- moved C13 14.6 mm to (73.0, 71.5)
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Connections:
- U1 pad 46: unconnected-(U1-PB10-Pad46) -> SPI2_SCK
- U1 pad 68: SPI2_SCK -> unconnected-(U1-PA9-Pad68)
Routing:
- net GND: track 72.7 -> 519.6 mm, vias 4 -> 27
- net 3.3V: track 9.12 -> 276.6 mm, vias 0 -> 19
- net 5V: track 20.0 -> 90.6 mm, vias 0 -> 5
- net Net-(J2-Pin_3): track 0.00 -> 58.1 mm, vias 0 -> 2
- net Net-(J2-Pin_2): track 0.00 -> 55.1 mm, vias 0 -> 2
- net D+: track 0.00 -> 51.4 mm
- net D-: track 0.00 -> 51.4 mm
- net PWM4: track 0.00 -> 46.9 mm
- net PYRO_3: track 11.2 -> 57.7 mm, vias 2 -> 6
- net PWM3: track 0.00 -> 42.1 mm
- net PYRO_2: track 6.09 -> 48.1 mm, vias 0 -> 4
- net PWM2: track 0.00 -> 37.3 mm
- net SPI4_NSS: track 0.00 -> 36.8 mm, vias 0 -> 1
- net LIPO_HIGH: track 47.1 -> 81.5 mm, vias 0 -> 3
- net PWM1: track 0.00 -> 32.5 mm
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Other:
- board size 50 x 77 mm -> 50 x 87 mm

Commit message: silkscreen
Other:
- board text added: "Ahsan Ahmed © 2026"
- board text added: "UltraHawk rev1"

Commit message: DRC fixes
Routing:
- net GND: track 519.6 -> 532.9 mm
- net 3.3V: track 276.6 -> 275.8 mm

Commit message: Journal Update
Parts:
- added C21: 100n, Capacitor_SMD:C_0805_2012Metric, F.Cu at (53.9, 100.5)
- C14: value C -> 1u
- C22: value 100n -> 1uf
- FB1: footprint Resistor_SMD:R_0805_2012Metric -> Resistor_SMD:R_0603_1608Metric_Pad0.98x0.95mm_HandSolder
- L1: footprint Inductor_SMD:L_0805_2012Metric -> easyeda2kicad:IND-SMD_L5.8-W5.2
- moved L1 18.1 mm to (77.8, 121.3)
Connections:
- U6 pad 5: Net-(U6-EN) -> LIPO_HIGH
Routing:
- net Net-(U6-SW): track 6.01 -> 26.1 mm, vias 0 -> 3
- net 5V: track 90.6 -> 87.6 mm, vias 5 -> 6
- net 3.3V: track 275.8 -> 278.1 mm
- net LIPO_HIGH: track 81.4 -> 83.6 mm
- net GND: track 532.9 -> 535.1 mm, vias 27 -> 28

Commit message: Journal Update
Parts:
- moved C21 0.20 mm to (53.9, 100.7)
- moved L1 0.20 mm to (78.0, 121.3)
Routing:
- net Net-(U6-EN): track 3.76 -> 0.00 mm
- net LIPO_HIGH: track 83.6 -> 84.3 mm
Changed lines of the file:
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@@
 	(footprint "Capacitor_SMD:C_0805_2012Metric"
 		(layer "F.Cu")
-		(at 53.85 100.5 180)
+		(at 53.85 100.7 180)
 		(descr "Capacitor SMD 0805 (2012 Metric), square (rectangular) end terminal, IPC-7351 nominal, (Body size source: IPC-SM-782 page 76, https://www.pcb-3d.com/wordpress/wp-content/uploads/ipc-sm-782a_amendment_1_and_2.pdf, https://docs.google.com/spreadsheets/d/1BsfQQcO9C6DZCsRaXUlFlo91Tg2WpOkGARC1WS5S8t0/edit?usp=sharing)")
 		(tags "capacitor")
@@
 	(footprint "easyeda2kicad:IND-SMD_L5.8-W5.2"
 		(layer "F.Cu")
-		(at 77.8 121.3 180)
+		(at 78 121.3 180)
 		(property "Reference" "L1"
 			(at 0 -4 180)
@@
 				(font
 					(size 1.27 1.27)
+					(thickness 0.15)
 				)
 			)
@@
 	)
 	(segment
+		(start 81.3625 137)
+		(end 80.700001 137)
+		(width 0.2)
+		(layer "F.Cu")
+		(net "LIPO_HIGH")
+	)
+	(segment
 		(start 95.6 121.1)
 		(end 95.6 128.4)
@@
 	)
 	(segment
-		(start 81.3625 137)
-		(end 80.700001 137)
-		(width 0.2)
-		(layer "F.Cu")
-		(net "Net-(U6-EN)")
-	)
-	(segment
-		(start 80.700001 137)
-		(end 80.2 137.500001)
-		(width 0.2)
-		(layer "F.Cu")
-		(net "Net-(U6-EN)")
-	)
-	(segment
-		(start 80.2 137.500001)
-		(end 80.2 139.8875)
-		(width 0.2)
-		(layer "F.Cu")
-		(net "Net-(U6-EN)")
-	)
-	(segment
